File: Telemetry_KiCAD_Project/Telemetry_KiCAD_Project.sch (KiCad schematic (older format))
At the start: 2 parts

Commit message: Included Amplifier, New Transceivers, Duplexer, and 37 Pin DSUB
Still want to replace the microcontroller, will happen in next commit
Parts:
- removed J?: CONN_06X2PTH_FEMALE, 2X6, symbol SparkFun-Connectors:CONN_06X2PTH_FEMALE
- removed J?: ARM 10 Pin, 2X5-RA, symbol SparkFun-Connectors:CONN_05X2RA
- added J?: Conn_Coaxial, symbol Connector:Conn_Coaxial
Connections:
- net labels added: RX_SCL, RX_SDI, RX_SDO, TX_SCL, TX_SDI, TX_SDO
- net labels removed: +3.3V, +5V, EXT_SCL, EXT_SDA, NRST, SWCLK, SWDIO
- wire segments 12 -> 31
- no-connect marks 3 -> 0
