File: Telemetry_KiCAD_Project/MCU_L552CC.sch (KiCad schematic (older format))
At the start: 13 parts

Commit message: Added USB ESD, relocated Debug pins
Connections:
- net DEBUG_SWCLK: now also U?.37 (PA14); no longer U?.34 (PA13)
- net DEBUG_SWDIO: now also U?.34 (PA13); no longer U?.26 (PB13)
- net EXT_INT1: now reaches U?.18 (PB0)
- new net EXT_INT2: U?.26 (PB13)
Changed lines of the file:
@@
 $Descr A4 11693 8268
 encoding utf-8
-Sheet 7 7
+Sheet 7 8
 Title ""
 Date ""
@@
 Text HLabel 5550 4750 0    50   Input ~ 0
 SPI2_MOSI
-Text HLabel 5550 4550 0    50   Input ~ 0
+Text HLabel 6750 4550 2    50   Input ~ 0
 DEBUG_SWDIO
 Text HLabel 5550 4150 0    50   Input ~ 0
@@
 Text HLabel 5550 3550 0    50   Input ~ 0
 SPI3_SCK
-Text HLabel 6750 4550 2    50   Input ~ 0
+Text HLabel 6750 4650 2    50   Input ~ 0
 DEBUG_SWCLK
 Text HLabel 6750 4450 2    50   Input ~ 0
@@
 Text Notes 3800 1350 0    100  ~ 0
 Microcontroller Chip
+Text HLabel 5550 3250 0    50   Input ~ 0
+EXT_INT1
+Text HLabel 5550 4550 0    50   Input ~ 0
+EXT_INT2
 $EndSCHEMATC

Commit message: Added chip select functions for RX and TX chips
The Si4463 datasheet mentions that some parameters can be quickly accessed if the chip select line is toggled
Connections:
- net ABORT_2: now also U?.15 (PA5); no longer U?.14 (PA4)
- net ~SPI2_CS: now reaches U?.25 (PB12)
- new net ~SPI3_CS: U?.14 (PA4)
Changed lines of the file:
@@
 Text HLabel 5550 3950 0    50   Input ~ 0
 I2C1_EN
-Text HLabel 6750 3550 2    50   Input ~ 0
-ABORT_1
-Text HLabel 6750 3650 2    50   Input ~ 0
-ABORT_2
 Text Notes 750  1000 0    100  ~ 0
 Microcontroller\nInput Power Filtering
@@
 Text HLabel 5550 4550 0    50   Input ~ 0
 EXT_INT2
+Text HLabel 6750 3750 2    50   Input ~ 0
+ABORT_2
+Text HLabel 6750 3550 2    50   Input ~ 0
+ABORT_1
+Text HLabel 5550 4450 0    50   Input ~ 0
+~SPI2_CS
+Text HLabel 6750 3650 2    50   Input ~ 0
+~SPI3_CS
 $EndSCHEMATC
