File: Telemetry_KiCAD_Project/Telemetry_KiCAD_Project.kicad_pcb (KiCad board)
At the start: 4 copper layers, 80 x 87.3 mm, 62 parts, among them J1 50Ω SMA Connector, J2 DB37_Male, J3 10118192-0001LF, U1 RSD-897.500-942.500-1612-TR, U2 Si4463, U3 ADL5521, U4 Si4463, U5 STM32L562VET, U6 LM317T, U7 USBLC6-2SC6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

Commit message: PCB Layout Progress
Routing:
- net (no net): track 6.23 -> 7.10 mm, vias 0 -> 1
- net GND: track 71.3 -> 70.6 mm, vias 37 -> 36
Changed lines of the file:
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@@
     (thickness 1.6)
     (drawings 17)
-    (tracks 669)
+    (tracks 670)
     (zones 0)
     (modules 62)
@@
   (segment (start 184.2 93.7) (end 185.2 94.7) (width 0.3) (layer Gnd.Cu) (net 0))
   (segment (start 182.5 93.7) (end 184.2 93.7) (width 0.3) (layer Gnd.Cu) (net 0))
+  (via (at 161.6 71.55) (size 0.8) (drill 0.4) (layers F.Cu B.Cu) (net 0))
+  (segment (start 161.55 71.6) (end 161.6 71.55) (width 0.25) (layer F.Cu) (net 0))
+  (segment (start 160.75 71.6) (end 161.55 71.6) (width 0.25) (layer F.Cu) (net 0))
+  (via (at 158.25 71.55) (size 0.8) (drill 0.4) (layers F.Cu B.Cu) (net 2))
+  (segment (start 159.25 71.55) (end 158.25 71.55) (width 0.25) (layer F.Cu) (net 2))
   (via (at 159.7 70.05) (size 0.8) (drill 0.4) (layers F.Cu B.Cu) (net 2))
   (segment (start 160 70.35) (end 159.7 70.05) (width 0.25) (layer F.Cu) (net 2))
@@
   (segment (start 160.55 72.67) (end 160.6 72.72) (width 0.25) (layer F.Cu) (net 2))
   (segment (start 159.4 72.72) (end 157.46 74.66) (width 0.25) (layer F.Cu) (net 2))
-  (segment (start 159.4 72.1) (end 158.55 72.1) (width 0.25) (layer F.Cu) (net 2))
   (segment (start 159.4 71.55) (end 159.4 72.1) (width 0.25) (layer F.Cu) (net 2))
-  (via (at 158.55 72.1) (size 0.8) (drill 0.4) (layers F.Cu B.Cu) (net 2))
   (segment (start 159.4 72.1) (end 159.4 72.72) (width 0.25) (layer F.Cu) (net 2))
-  (via (at 161.45 72.2) (size 0.8) (drill 0.4) (layers F.Cu B.Cu) (net 2))
-  (segment (start 160.55 72.2) (end 161.45 72.2) (width 0.25) (layer F.Cu) (net 2))
   (segment (start 160.55 71.65) (end 160.55 72.2) (width 0.25) (layer F.Cu) (net 2))
   (segment (start 160.55 72.2) (end 160.55 72.67) (width 0.25) (layer F.Cu) (net 2))
