File: Hardware/Telemetry_KiCAD_Project.sch (KiCad schematic (older format))
At the start: 1 part, among them J1 50Ω SMA Connector

Commit message: Fixed merge mistakes between branches
Parts:
- added TP1, TP10, TP11, TP12, TP13, TP14, TP15, TP16, TP17, TP18, TP19, TP2, TP20, TP21, TP22, TP23, TP24, TP25, TP3, TP4, TP5, TP6, TP7, TP8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: TestPoint_Small, TestPoint:TestPoint_Loop_D1.80mm_Drill1.0mm_Beaded, symbol Connector:TestPoint_Small
Connections:
- wire segments 45 -> 70
Other:
- moved on the sheet: J1
