File: Hardware/Telemetry_KiCAD_Project.kicad_sch (KiCad schematic)
At the start: 3 parts, among them J1 TX SPI Debug, J2 RX SPI Debug, J3 Amphenol 132134 SMA Connector

Commit message: Adapted layout to different linear regulator for USB
Other:
- sheet MCU_L562VE ports: added USB_D+, USB_D-; removed USB_DM, USB_DP
Changed lines of the file:
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@@
       (effects (font (size 1.27 1.27)) (justify left))
     )
-    (pin "USB_DP" input (at 104.14 113.03 0)
-      (effects (font (size 1.27 1.27)) (justify right))
-    )
-    (pin "USB_DM" input (at 104.14 116.84 0)
+    (pin "USB_D+" input (at 104.14 113.03 0)
+      (effects (font (size 1.27 1.27)) (justify right))
+    )
+    (pin "USB_D-" input (at 104.14 116.84 0)
       (effects (font (size 1.27 1.27)) (justify right))
     )
@@
       (reference "#PWR021") (unit 1) (value "+5V") (footprint "")
     )
-    (path "/00000000-0000-0000-0000-000061a2ed84/00000000-0000-0000-0000-000061a45748"
-      (reference "#PWR022") (unit 1) (value "GND") (footprint "")
-    )
-    (path "/00000000-0000-0000-0000-000061a2ed84/00000000-0000-0000-0000-000061a459ef"
-      (reference "#PWR023") (unit 1) (value "GND") (footprint "")
-    )
     (path "/00000000-0000-0000-0000-000061a2ed84/00000000-0000-0000-0000-000061a3a807"
       (reference "#PWR024") (unit 1) (value "+3.3V") (footprint "")
@@
       (reference "#PWR0105") (unit 1) (value "GND") (footprint "")
     )
+    (path "/00000000-0000-0000-0000-000061a2ed84/62c214f9-69e5-4473-9247-07d67610f672"
+      (reference "#PWR0106") (unit 1) (value "GND") (footprint "")
+    )
+    (path "/00000000-0000-0000-0000-000061a2ed84/55982482-7869-4778-ab3f-3dec7bf36852"
+      (reference "#PWR0107") (unit 1) (value "GND") (footprint "")
+    )
+    (path "/00000000-0000-0000-0000-000061a2ed84/9241d27b-cee7-4065-b480-439c4f4d64ef"
+      (reference "#PWR0108") (unit 1) (value "GND") (footprint "")
+    )
     (path "/00000000-0000-0000-0000-000061a0416a/00000000-0000-0000-0000-0000619f8bd8"
       (reference "C1") (unit 1) (value "100pF") (footprint "Capacitor_SMD:C_0402_1005Metric")
@@
       (reference "U3") (unit 1) (value "RSD-897.500-942.500-1612-TR") (footprint "RDT_Custom_Footprints:RSD-897.500-942.500-1612-TR")
     )
-    (path "/00000000-0000-0000-0000-000061a2ed84/00000000-0000-0000-0000-000061a380e7"
-      (reference "U4") (unit 1) (value "LM317T") (footprint "Package_TO_SOT_SMD:TSOT-23")
+    (path "/00000000-0000-0000-0000-000061a2ed84/9a5e7e18-5e99-4a60-ba18-d8e2fceef78a"
+      (reference "U4") (unit 1) (value "LP38692MPX-ADJ") (footprint "Package_TO_SOT_SMD:SOT-223-5")
     )
     (path "/00000000-0000-0000-0000-000061a2ed84/00000000-0000-0000-0000-000061a51e77"

Commit message: Adjusted 5V lines, corrected ground fences, added cutout for USB connector
Parts:
- J3: value Amphenol 132134 SMA Connector -> Right Angle SMA Female; footprint Connector_Coaxial:SMA_Amphenol_132134-11_Vertical -> Connector_Coaxial:SMA_Molex_73251-2200_Horizontal
Changed lines of the file:
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@@
       (effects (font (size 1.27 1.27)) (justify left))
     )
-    (property "Value" "Amphenol 132134 SMA Connector" (id 1) (at 248.92 90.5764 0)
-      (effects (font (size 1.27 1.27)) (justify left))
-    )
-    (property "Footprint" "Connector_Coaxial:SMA_Amphenol_132134-11_Vertical" (id 2) (at 246.38 87.63 0)
+    (property "Value" "Right Angle SMA Female" (id 1) (at 248.92 90.5764 0)
+      (effects (font (size 1.27 1.27)) (justify left))
+    )
+    (property "Footprint" "Connector_Coaxial:SMA_Molex_73251-2200_Horizontal" (id 2) (at 246.38 87.63 0)
       (effects (font (size 1.27 1.27)) hide)
     )
@@
     )
     (path "/00000000-0000-0000-0000-000061a2ed84/00000000-0000-0000-0000-000061a3a235"
-      (reference "D1") (unit 1) (value "D_Schottky_Small") (footprint "Diode_SMD:D_0603_1608Metric_Pad1.05x0.95mm_HandSolder")
+      (reference "D1") (unit 1) (value "D_Schottky_Small") (footprint "Diode_SMD:D_0805_2012Metric_Pad1.15x1.40mm_HandSolder")
     )
     (path "/00000000-0000-0000-0000-000061a107a5/00000000-0000-0000-0000-000061eaa754"
@@
     )
     (path "/00000000-0000-0000-0000-0000619fd788"
-      (reference "J3") (unit 1) (value "Amphenol 132134 SMA Connector") (footprint "Connector_Coaxial:SMA_Amphenol_132134-11_Vertical")
+      (reference "J3") (unit 1) (value "Right Angle SMA Female") (footprint "Connector_Coaxial:SMA_Molex_73251-2200_Horizontal")
     )
     (path "/00000000-0000-0000-0000-000061a2ed84/00000000-0000-0000-0000-000061a3682f"

Commit message: Updated schematic labels, Version 2.0.0
Other:
- company: Missouri S&T Rocket Design Team '21 (Thomas Francois) -> When HAMs Fly Senior Design Team
Changed lines of the file:
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@@
   (title_block
     (title "Telemetry PCB Schematic")
-    (date "2021-10-01")
-    (rev "v1.0.1")
-    (company "Missouri S&T Rocket Design Team '21 (Thomas Francois)")
+    (date "2022-03-24")
+    (rev "v2.0.0")
+    (company "When HAMs Fly Senior Design Team")
     (comment 1 "https://github.com/MSTRocketDesignTeam/Avionics-Telemetry-PCB")
-    (comment 2 "Intended as initial pre-production design")
+    (comment 2 "Board Revision 2")
     (comment 3 "Schematic depicting logical connections between components")
   )
