File: Hardware/Telemetry_KiCAD_Project.kicad_sch (KiCad schematic)
At the start: 3 parts, among them J1 TX SPI Debug, J2 RX SPI Debug, J3 Right Angle SMA Female

Commit message: Added more JLC part numbers and added missing voltage regulator connection
Parts:
- J3: LCSC (none) -> C429844
Changed lines of the file:
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@@
+      (effects (font (size 1.27 1.27)) hide)
+    )
+    (property "LCSC" "C429844" (id 4) (at 246.38 87.63 0)
       (effects (font (size 1.27 1.27)) hide)
     )

Commit message: Added resistor that was missing, connected a resistor that was floating, and updated LCSC numbers
Parts:
- J3: LCSC C429844 -> C3174425
Changed lines of the file:
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@@
       (effects (font (size 1.27 1.27)) hide)
     )
-    (property "LCSC" "C429844" (id 4) (at 246.38 87.63 0)
+    (property "LCSC" "C3174425" (id 4) (at 246.38 87.63 0)
       (effects (font (size 1.27 1.27)) hide)
     )
@@
     )
     (path "/00000000-0000-0000-0000-000061a107a5/1e76e978-f957-40c0-bfb3-aaa084b976c8"
-      (reference "R11") (unit 1) (value "4.7k") (footprint "Resistor_SMD:R_0603_1608Metric_Pad1.05x0.95mm_HandSolder")
+      (reference "R11") (unit 1) (value "4.7k") (footprint "Resistor_SMD:R_0603_1608Metric_Pad0.98x0.95mm_HandSolder")
     )
     (path "/00000000-0000-0000-0000-000061a107a5/3376bd56-9efd-4f2b-852a-e2dafccb6289"
