File: Hardware/COMPONENT_SHEETS/RSD_Duplexer.kicad_sch (KiCad schematic)
At the start: 1 part, among them U3 RSD-897.500-942.500-1612-TR

Commit message: Updated schematic labels, Version 2.0.0
Other:
- company: (none) -> When HAMs Fly Senior Design Team
- title: (none) -> Duplexer Network
Changed lines of the file:
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@@
 (kicad_sch (version 20211123) (generator eeschema)
   (paper "A4")
+  (title_block
+    (title "Duplexer Network")
+    (date "2022-03-24")
+    (rev "v2.0.0")
+    (company "When HAMs Fly Senior Design Team")
+    (comment 1 "https://github.com/MSTRocketDesignTeam/Avionics-Telemetry-PCB")
+    (comment 2 "Board Revision 2")
+    (comment 3 "Schematic depicting logical connections between components")
+  )
   (junction (at 158.75 102.87) (diameter 0) (color 0 0 0 0)
   )

Commit message: Updated LCSC numbers and production files
Parts:
- U3: LCSC (none) -> C3271762
Changed lines of the file:
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@@
+      (effects (font (size 1.27 1.27)) hide)
+    )
+    (property "LCSC" "C3271762" (id 4) (at 135.89 92.71 0)
       (effects (font (size 1.27 1.27)) hide)
     )
