File: Hardware/COMPONENT_SHEETS/MCU_L562VE.kicad_sch (KiCad schematic)
At the start: 33 parts, among them SW1 MCU Reset, U7 STM32L562VET6Q, Y3 32MHz

Commit message: Added more JLC part numbers and added missing voltage regulator connection
Parts:
- U7: LCSC (none) -> C1236652
Changed lines of the file:
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@@
     )
     (property "Description" "Microcontroller" (id 4) (at 100.33 100.33 0))
+    (property "LCSC" "C1236652" (id 5) (at 100.33 29.21 0)
+      (effects (font (size 1.27 1.27)) hide)
+    )
     (pin "1")
     (pin "10")

Commit message: Updated LCSC numbers and production files
Parts:
- C24, C25: LCSC C22397 -> C400083
- D3, D5: LCSC C165982 -> C138548
- Y3: LCSC (none) -> C1986810
Changed lines of the file:
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@@
       (effects (font (size 1.27 1.27)) hide)
     )
-    (property "LCSC" "C22397" (id 4) (at 21.59 83.82 0)
+    (property "LCSC" "C400083" (id 4) (at 21.59 83.82 0)
       (effects (font (size 1.27 1.27)) hide)
     )
@@
       (effects (font (size 1.27 1.27)) hide)
     )
-    (property "LCSC" "C22397" (id 4) (at 31.75 83.82 0)
+    (property "LCSC" "C400083" (id 4) (at 31.75 83.82 0)
       (effects (font (size 1.27 1.27)) hide)
     )
@@
     )
     (property "Datasheet" "~" (id 3) (at 26.67 78.74 0)
+      (effects (font (size 1.27 1.27)) hide)
+    )
+    (property "LCSC" "C1986810" (id 4) (at 26.67 78.74 0)
       (effects (font (size 1.27 1.27)) hide)
     )
@@
       (effects (font (size 1.27 1.27)) hide)
     )
-    (property "LCSC" " C165982 " (id 4) (at 44.45 120.65 90)
+    (property "LCSC" "C138548" (id 4) (at 44.45 120.65 90)
       (effects (font (size 1.27 1.27)) hide)
     )
@@
       (effects (font (size 1.27 1.27)) hide)
     )
-    (property "LCSC" " C165982 " (id 4) (at 29.21 120.65 90)
+    (property "LCSC" "C138548" (id 4) (at 29.21 120.65 90)
       (effects (font (size 1.27 1.27)) hide)
     )

Commit message: Added resistor that was missing, connected a resistor that was floating, and updated LCSC numbers
Parts:
- R11: footprint Resistor_SMD:R_0603_1608Metric_Pad1.05x0.95mm_HandSolder -> Resistor_SMD:R_0603_1608Metric_Pad0.98x0.95mm_HandSolder
Changed lines of the file:
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@@
     (property "Reference" "R11" (id 0) (at 245.745 79.375 0))
     (property "Value" "4.7k" (id 1) (at 245.745 76.835 0))
-    (property "Footprint" "Resistor_SMD:R_0603_1608Metric_Pad1.05x0.95mm_HandSolder" (id 2) (at 242.57 78.105 0)
+    (property "Footprint" "Resistor_SMD:R_0603_1608Metric_Pad0.98x0.95mm_HandSolder" (id 2) (at 242.57 78.105 0)
       (effects (font (size 1.27 1.27)) hide)
     )
