File: Hardware/COMPONENT_SHEETS/ADL_Amplifier.kicad_sch (KiCad schematic)
At the start: 6 parts, among them U2 ADL5521

Commit message: Updated schematic labels, Version 2.0.0
Other:
- company: (none) -> When HAMs Fly Senior Design Team
- title: (none) -> ADL5521 Amplifier Network
Changed lines of the file:
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@@
 (kicad_sch (version 20211123) (generator eeschema)
   (paper "A4")
+  (title_block
+    (title "ADL5521 Amplifier Network")
+    (date "2022-03-24")
+    (rev "v2.0.0")
+    (company "When HAMs Fly Senior Design Team")
+    (comment 1 "https://github.com/MSTRocketDesignTeam/Avionics-Telemetry-PCB")
+    (comment 2 "Board Revision 2")
+    (comment 3 "Schematic depicting logical connections between components")
+  )
   (junction (at 81.28 78.74) (diameter 0) (color 0 0 0 0)
   )

Commit message: Updated LCSC numbers and production files
Parts:
- U2: LCSC (none) -> C657768
Changed lines of the file:
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@@
+      (effects (font (size 1.27 1.27)) hide)
+    )
+    (property "LCSC" "C657768" (id 4) (at 97.79 72.39 0)
       (effects (font (size 1.27 1.27)) hide)
     )

Commit message: Fixed incorrect LCSC numbers
Parts:
- C12: LCSC C123475 -> C307331
Changed lines of the file:
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@@
       (effects (font (size 1.27 1.27)) hide)
     )
-    (property "LCSC" "C123475" (id 4) (at 120.65 53.34 90)
+    (property "LCSC" "C307331" (id 4) (at 120.65 53.34 90)
       (effects (font (size 1.27 1.27)) hide)
     )
