File: Hardware/COMPONENT_SHEETS/DSUB-37_Male.kicad_sch (KiCad schematic)
At the start: 1 part, among them J5 DB37_Male_MountingHoles

Commit message: Updated schematic labels, Version 2.0.0
Other:
- company: (none) -> When HAMs Fly Senior Design Team
- title: (none) -> DSUB Connector
Changed lines of the file:
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@@
 (kicad_sch (version 20211123) (generator eeschema)
   (paper "A4")
+  (title_block
+    (title "DSUB Connector")
+    (date "2022-03-24")
+    (rev "v2.0.0")
+    (company "When HAMs Fly Senior Design Team")
+    (comment 1 "https://github.com/MSTRocketDesignTeam/Avionics-Telemetry-PCB")
+    (comment 2 "Board Revision 2")
+    (comment 3 "Schematic depicting logical connections between components")
+  )
   (wire (pts (xy 189.23 120.65) (xy 189.23 119.38))
     (stroke (width 0) (type default) (color 0 0 0 0))
