File: Hardware/COMPONENT_SHEETS/Si4463_TX.kicad_sch (KiCad schematic)
At the start: 16 parts, among them U6 Si4463, Y2 32MHz

Commit message: Updated schematic labels, Version 2.0.0
Other:
- company: (none) -> When HAMs Fly Senior Design Team
- title: (none) -> SI4463 Transmit Network
Changed lines of the file:
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@@
 (kicad_sch (version 20211123) (generator eeschema)
   (paper "A4")
+  (title_block
+    (title "SI4463 Transmit Network")
+    (date "2022-03-24")
+    (rev "v2.0.0")
+    (company "When HAMs Fly Senior Design Team")
+    (comment 1 "https://github.com/MSTRocketDesignTeam/Avionics-Telemetry-PCB")
+    (comment 2 "Board Revision 2")
+    (comment 3 "Schematic depicting logical connections between components")
+  )
   (junction (at 120.65 93.98) (diameter 0) (color 0 0 0 0)
   )

Commit message: Added more JLC part numbers and added missing voltage regulator connection
Parts:
- U6: LCSC (none) -> C476202
Changed lines of the file:
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@@
+      (effects (font (size 1.27 1.27)) hide)
+    )
+    (property "LCSC" "C476202" (id 5) (at 156.21 92.71 0)
       (effects (font (size 1.27 1.27)) hide)
     )

Commit message: Updated LCSC numbers and production files
Parts:
- C16, C18: LCSC C22397 -> C400083
- Y2: LCSC (none) -> C1986810
Changed lines of the file:
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@@
       (effects (font (size 1.27 1.27)) hide)
     )
-    (property "LCSC" "C22397" (id 4) (at 120.65 99.06 0)
+    (property "LCSC" "C400083" (id 4) (at 120.65 99.06 0)
       (effects (font (size 1.27 1.27)) hide)
     )
@@
       (effects (font (size 1.27 1.27)) hide)
     )
-    (property "LCSC" "C22397" (id 4) (at 130.81 99.06 0)
+    (property "LCSC" "C400083" (id 4) (at 130.81 99.06 0)
       (effects (font (size 1.27 1.27)) hide)
     )
@@
       (effects (font (size 1.27 1.27)) hide)
     )
+    (property "LCSC" "C1986810" (id 4) (at 125.73 93.98 0)
+      (effects (font (size 1.27 1.27)) hide)
+    )

Commit message: Fixed incorrect LCSC numbers
Parts:
- L6: LCSC C27147 -> C22726
Changed lines of the file:
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@@
       (effects (font (size 1.27 1.27)) hide)
     )
-    (property "LCSC" "C27147" (id 4) (at 171.45 73.66 0)
+    (property "LCSC" "C22726" (id 4) (at 171.45 73.66 0)
       (effects (font (size 1.27 1.27)) hide)
     )

Commit message: Updated LCSC numbers and cleaned up routing
Parts:
- C16, C18: LCSC C400083 -> C123555
Changed lines of the file:
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@@
       (effects (font (size 1.27 1.27)) hide)
     )
-    (property "LCSC" "C400083" (id 4) (at 120.65 99.06 0)
+    (property "LCSC" "C123555" (id 4) (at 120.65 99.06 0)
       (effects (font (size 1.27 1.27)) hide)
     )
@@
       (effects (font (size 1.27 1.27)) hide)
     )
-    (property "LCSC" "C400083" (id 4) (at 130.81 99.06 0)
+    (property "LCSC" "C123555" (id 4) (at 130.81 99.06 0)
       (effects (font (size 1.27 1.27)) hide)
     )
