File: Hardware/COMPONENT_SHEETS/Si4463_RX.kicad_sch (KiCad schematic)
At the start: 15 parts, among them U1 Si4463, Y1 32MHz

Commit message: Updated schematic labels, Version 2.0.0
Other:
- company: (none) -> When HAMs Fly Senior Design Team
- title: (none) -> SI4463 Receive Network
Changed lines of the file:
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@@
 (kicad_sch (version 20211123) (generator eeschema)
   (paper "A4")
+  (title_block
+    (title "SI4463 Receive Network")
+    (date "2022-03-24")
+    (rev "v2.0.0")
+    (company "When HAMs Fly Senior Design Team")
+    (comment 1 "https://github.com/MSTRocketDesignTeam/Avionics-Telemetry-PCB")
+    (comment 2 "Board Revision 2")
+    (comment 3 "Schematic depicting logical connections between components")
+  )
   (junction (at 213.36 87.63) (diameter 0) (color 0 0 0 0)
   )

Commit message: Added more JLC part numbers and added missing voltage regulator connection
Parts:
- U1: LCSC (none) -> C476202
Changed lines of the file:
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@@
+      (effects (font (size 1.27 1.27)) hide)
+    )
+    (property "LCSC" "C476202" (id 5) (at 156.21 92.71 0)
       (effects (font (size 1.27 1.27)) hide)
     )

Commit message: Updated LCSC numbers and production files
Parts:
- C2, C4: LCSC C22397 -> C400083
- Y1: LCSC (none) -> C1986810
Changed lines of the file:
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@@
       (effects (font (size 1.27 1.27)) hide)
     )
-    (property "LCSC" "C22397" (id 4) (at 121.92 99.06 0)
+    (property "LCSC" "C400083" (id 4) (at 121.92 99.06 0)
       (effects (font (size 1.27 1.27)) hide)
     )
@@
       (effects (font (size 1.27 1.27)) hide)
     )
-    (property "LCSC" "C22397" (id 4) (at 132.08 99.06 0)
+    (property "LCSC" "C400083" (id 4) (at 132.08 99.06 0)
       (effects (font (size 1.27 1.27)) hide)
     )
@@
       (effects (font (size 1.27 1.27)) hide)
     )
+    (property "LCSC" "C1986810" (id 4) (at 127 93.98 0)
+      (effects (font (size 1.27 1.27)) hide)
+    )

Commit message: Updated LCSC and production files
Parts:
- C8: LCSC (none) -> C1550
Changed lines of the file:
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@@
+      (effects (font (size 1.27 1.27)) hide)
+    )
+    (property "LCSC" " C1550 " (id 4) (at 199.39 87.63 90)
       (effects (font (size 1.27 1.27)) hide)
     )

Commit message: Updated LCSC numbers and cleaned up routing
Parts:
- C2, C4: LCSC C400083 -> C123555
Changed lines of the file:
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@@
       (effects (font (size 1.27 1.27)) hide)
     )
-    (property "LCSC" "C400083" (id 4) (at 121.92 99.06 0)
+    (property "LCSC" "C123555" (id 4) (at 121.92 99.06 0)
       (effects (font (size 1.27 1.27)) hide)
     )
@@
       (effects (font (size 1.27 1.27)) hide)
     )
-    (property "LCSC" "C400083" (id 4) (at 132.08 99.06 0)
+    (property "LCSC" "C123555" (id 4) (at 132.08 99.06 0)
       (effects (font (size 1.27 1.27)) hide)
     )

Commit message: Updated LCSC numbers, updated BOM file, added power LED.
Parts:
- C6: LCSC C318583 -> C115630
Changed lines of the file:
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@@
       (effects (font (size 1.27 1.27)) hide)
     )
-    (property "LCSC" "C318583" (id 4) (at 176.53 99.06 0)
+    (property "LCSC" "C115630" (id 4) (at 176.53 99.06 0)
       (effects (font (size 1.27 1.27)) hide)
     )
